Commit message: Update joint name - joint_1 --> joint_a1

File: create_kr240_robot_description/urdf/kr240_r3330_macro.xacro (robot description, xacro)
@@ -146,5 +146,5 @@
     <!-- JOINTS -->
     <!-- joint 1 (A1) -->
-    <joint name="${prefix}joint_1" type="revolute">
+    <joint name="${prefix}joint_a1" type="revolute">
       <axis xyz="0.0 0.0 1.0"/>
       <child link="${prefix}link_1"/>
@@ -154,5 +154,5 @@
     </joint>
     <!-- joint 2 (A2) -->
-    <joint name="${prefix}joint_2" type="revolute">
+    <joint name="${prefix}joint_a2" type="revolute">
       <axis xyz="0.0 0.0 1.0"/>
       <child link="${prefix}link_2"/>
@@ -162,5 +162,5 @@
     </joint>
     <!-- joint 3 (A3) -->
-    <joint name="${prefix}joint_3" type="revolute">
+    <joint name="${prefix}joint_a3" type="revolute">
       <axis xyz="0.0 0.0 1.0"/>
       <child link="${prefix}link_3"/>
@@ -170,5 +170,5 @@
     </joint>
     <!-- joint 4 (A4) -->
-    <joint name="${prefix}joint_4" type="revolute">
+    <joint name="${prefix}joint_a4" type="revolute">
       <axis xyz="0.0 0.0 1.0"/>
       <child link="${prefix}link_4"/>
@@ -178,5 +178,5 @@
     </joint>
     <!-- joint 5 (A5) -->
-    <joint name="${prefix}joint_5" type="revolute">
+    <joint name="${prefix}joint_a5" type="revolute">
       <axis xyz="0.0 0.0 1.0"/>
       <child link="${prefix}link_5"/>
@@ -186,5 +186,5 @@
     </joint>
     <!-- joint 6 (A6) -->
-    <joint name="${prefix}joint_6" type="revolute">
+    <joint name="${prefix}joint_a6" type="revolute">
       <axis xyz="0.0 0.0 1.0"/>
       <child link="${prefix}link_6"/>
