Commit message: Fix Rail & Robot URDF

File: create_kr240_robot_description/urdf/kl4000_macro.xacro (robot description, xacro)
@@ -20,5 +20,5 @@
             <mesh filename="file://$(find create_kr240_robot_description)/meshes/kl4000/visual/KL4000_Rail.dae"/>
         </geometry>
-        <origin rpy="-3.141592653589793 0.0 -0.0" xyz="0.0 -4.898587196589413e-17 0.4"/>
+        <origin rpy="0.0 0.0 0.0" xyz="0.0 0.0 0.0"/>
       </visual>
     </link>
@@ -29,10 +29,10 @@
           <mesh filename="file://$(find create_kr240_robot_description)/meshes/kl4000/collision/KL4000_Carriage_Collision.stl"/>
         </geometry>
-        <origin rpy="0.0 0.0 0.0" xyz="0.0 0.0 0.0"/>
+        <origin rpy="0.0 0.0 3.14159" xyz="0.0 0.0 0.0"/>
       </collision>
       <inertial>
         <inertia ixx="14.5413" ixy="0.0" ixz="0.0" iyy="147.936" iyz="0.0" izz="151.0383"/>
         <mass value="4.476E2"/>
-        <origin rpy="0.0 0.0 0.0" xyz="0.0 0.0 0.0"/>
+        <origin rpy="0.0 0.0 3.14159" xyz="0.0 0.0 0.0"/>
       </inertial>
       <visual>
@@ -40,5 +40,5 @@
             <mesh filename="file://$(find create_kr240_robot_description)/meshes/kl4000/visual/KL4000_Carriage.dae"/>
         </geometry>
-        <origin rpy="0.0 0.0 0.0" xyz="0.0 0.0 0.0"/>
+        <origin rpy="0.0 0.0 3.14159" xyz="0.0 0.0 0.0"/>
       </visual>
     </link>
@@ -46,9 +46,9 @@
     <!-- JOINTS -->
     <!-- joint rail-carriage -->
-    <joint name="${prefix}rail-carriage" type="linear">
+    <joint name="${prefix}rail-carriage" type="prismatic">
       <axis xyz="1.0 0.0 0.0"/>
       <child link="${prefix}carriage"/>
-      <limit effort="1.44E4" lower="-5000.0" upper="1000.0" velocity="500"/>
-      <origin rpy="0.0 0.0 0.0" xyz="0.0 0.0 0.0"/>
+      <limit effort="1.44E4" lower="-4.0" upper="1.0" velocity="0.5"/>
+      <origin rpy="0.0 0.0 3.14159" xyz="1.0 0.0 0.689"/>
       <parent link="${prefix}rail"/>
     </joint>
@@ -57,5 +57,5 @@
     <joint name="${prefix}carriage-mount" type="fixed">
       <child link="${prefix}mount"/>
-      <origin rpy="0.0 0.0 0.0" xyz="0.0 0.0 0.0"/>
+      <origin rpy="0.0 0.0 3.14159" xyz="0.0 0.0 0.0"/>
       <parent link="${prefix}carriage"/>
     </joint>

File: create_kr240_robot_description/urdf/kr240_kl4000.urdf.xacro (robot description, xacro)
@@ -4,10 +4,10 @@
     <xacro:include filename="$(find create_kr240_robot_description)/urdf/kr240_r3330_macro.xacro" />
     <xacro:include filename="$(find create_kr240_robot_description)/urdf/kl4000_macro.xacro" />
-    <xacro:kuka_kr240_r3330_robot prefix="${prefix}"/>
-    <xacro:kuka_kl4000_rail prefix="${prefix}"/>
-    <joint name="${prefix}carriage-robot" type="fixed">
-      <child link="${prefix}base"/>
+    <xacro:kuka_kr240_r3330_robot prefix=""/>
+    <xacro:kuka_kl4000_rail prefix=""/>
+    <joint name="$carriage-robot" type="fixed">
+      <child link="base_link"/>
       <origin rpy="0.0 0.0 0.0" xyz="0.0 0.0 0.0"/>
-      <parent link="${prefix}mount"/>
+      <parent link="mount"/>
     </joint>
 </robot>

File: create_kr240_robot_description/urdf/kr240_r3330_macro.xacro (robot description, xacro)
@@ -149,5 +149,5 @@
       <axis xyz="0.0 0.0 1.0"/>
       <child link="${prefix}link_1"/>
-      <limit effort="1.44E4" lower="-3.2288591125E0" upper="3.2288591125E0" velocity="1.7456E0"/>
+      <limit effort="1.44E4" lower="-2.87979E0" upper="2.87979E0" velocity="1.7456E0"/>
       <origin rpy="3.141592653589793 -0.0 0.0" xyz="0.0 0.0 0.4"/>
       <parent link="${prefix}base_link"/>
