Commit message: WIP

File: create_kr240_robot_description/urdf/kl4000_macro.xacro (robot description, xacro)
@@ -49,6 +49,6 @@
       <axis xyz="1.0 0.0 0.0"/>
       <child link="${prefix}carriage"/>
-      <limit effort="1.44E4" lower="-4.0" upper="1.0" velocity="0.5"/>
-      <origin rpy="0.0 0.0 3.14159" xyz="1.0 0.0 0.689"/>
+      <limit effort="1.44E4" lower="-5.0" upper="0.1" velocity="0.5"/>
+      <origin rpy="0.0 0.0 3.14159" xyz="0.1 0.0 0.689"/>
       <parent link="${prefix}rail"/>
     </joint>

File: create_kr240_robot_description/urdf/kr240_r3330_macro.ros2_control.xacro (robot description, xacro)
@@ -2,72 +2,70 @@
 <robot xmlns:xacro="http://www.ros.org/wiki/xacro">
   <xacro:macro name="kuka_kr240_r3330_ros2_control" params="prefix use_motion_primitives_driver:=^|true initial_positions:=${dict(joint_a1=0.0,joint_a2=-1.57,joint_a3=1.57,joint_a4=0.0,joint_a5=1.57,joint_a6=0.0)}">
-    <xacro:if value="${use_motion_primitives_driver}">
-      <joint name="${prefix}joint_a1">
-        <xacro:unless value="${use_motion_primitives_driver}">
-          <command_interface name="position">
-            <param name="min">-1</param>
-            <param name="max">1</param>
-          </command_interface>
-        </xacro:unless>
-        <state_interface name="position">
-          <param name="initial_value">${initial_positions['joint_a1']}</param>
-        </state_interface>
-      </joint>
-      <joint name="${prefix}joint_a2">
-        <xacro:unless value="${use_motion_primitives_driver}">
-          <command_interface name="position">
-            <param name="min">-1</param>
-            <param name="max">1</param>
-          </command_interface>
-        </xacro:unless>
-        <state_interface name="position">
-          <param name="initial_value">${initial_positions['joint_a2']}</param>
-        </state_interface>
-      </joint>
-      <joint name="${prefix}joint_a3">
-        <xacro:unless value="${use_motion_primitives_driver}">
-          <command_interface name="position">
-            <param name="min">-1</param>
-            <param name="max">1</param>
-          </command_interface>
-        </xacro:unless>
-        <state_interface name="position">
-          <param name="initial_value">${initial_positions['joint_a3']}</param>
-        </state_interface>
-      </joint>
-      <joint name="${prefix}joint_a4">
-        <xacro:unless value="${use_motion_primitives_driver}">
-          <command_interface name="position">
-            <param name="min">-1</param>
-            <param name="max">1</param>
-          </command_interface>
-        </xacro:unless>
-        <state_interface name="position">
-          <param name="initial_value">${initial_positions['joint_a4']}</param>
-        </state_interface>
-      </joint>
-      <joint name="${prefix}joint_a5">
-        <xacro:unless value="${use_motion_primitives_driver}">
-          <command_interface name="position">
-            <param name="min">-1</param>
-            <param name="max">1</param>
-          </command_interface>
-        </xacro:unless>
-        <state_interface name="position">
-          <param name="initial_value">${initial_positions['joint_a5']}</param>
-        </state_interface>
-      </joint>
-      <joint name="${prefix}joint_a6">
-        <xacro:unless value="${use_motion_primitives_driver}">
-          <command_interface name="position">
-            <param name="min">-1</param>
-            <param name="max">1</param>
-          </command_interface>
-        </xacro:unless>
-        <state_interface name="position">
-          <param name="initial_value">${initial_positions['joint_a6']}</param>
-        </state_interface>
-      </joint>
-    </xacro:if>
+    <joint name="${prefix}joint_a1">
+      <xacro:unless value="${use_motion_primitives_driver}">
+        <command_interface name="position">
+          <param name="min">-1</param>
+          <param name="max">1</param>
+        </command_interface>
+      </xacro:unless>
+      <state_interface name="position">
+        <param name="initial_value">${initial_positions['joint_a1']}</param>
+      </state_interface>
+    </joint>
+    <joint name="${prefix}joint_a2">
+      <xacro:unless value="${use_motion_primitives_driver}">
+        <command_interface name="position">
+          <param name="min">-1</param>
+          <param name="max">1</param>
+        </command_interface>
+      </xacro:unless>
+      <state_interface name="position">
+        <param name="initial_value">${initial_positions['joint_a2']}</param>
+      </state_interface>
+    </joint>
+    <joint name="${prefix}joint_a3">
+      <xacro:unless value="${use_motion_primitives_driver}">
+        <command_interface name="position">
+          <param name="min">-1</param>
+          <param name="max">1</param>
+        </command_interface>
+      </xacro:unless>
+      <state_interface name="position">
+        <param name="initial_value">${initial_positions['joint_a3']}</param>
+      </state_interface>
+    </joint>
+    <joint name="${prefix}joint_a4">
+      <xacro:unless value="${use_motion_primitives_driver}">
+        <command_interface name="position">
+          <param name="min">-1</param>
+          <param name="max">1</param>
+        </command_interface>
+      </xacro:unless>
+      <state_interface name="position">
+        <param name="initial_value">${initial_positions['joint_a4']}</param>
+      </state_interface>
+    </joint>
+    <joint name="${prefix}joint_a5">
+      <xacro:unless value="${use_motion_primitives_driver}">
+        <command_interface name="position">
+          <param name="min">-1</param>
+          <param name="max">1</param>
+        </command_interface>
+      </xacro:unless>
+      <state_interface name="position">
+        <param name="initial_value">${initial_positions['joint_a5']}</param>
+      </state_interface>
+    </joint>
+    <joint name="${prefix}joint_a6">
+      <xacro:unless value="${use_motion_primitives_driver}">
+        <command_interface name="position">
+          <param name="min">-1</param>
+          <param name="max">1</param>
+        </command_interface>
+      </xacro:unless>
+      <state_interface name="position">
+        <param name="initial_value">${initial_positions['joint_a6']}</param>
+      </state_interface>
+    </joint>
   </xacro:macro>
 </robot>

File: create_kr240_robot_description/urdf/kr240_r3330_macro.xacro (robot description, xacro)
@@ -32,5 +32,5 @@
       </collision>
       <inertial>
-        <inertia ixx="0.0" ixy="0.0" ixz="0.0" iyy="6.87109208044536E-31" iyz="0.0" izz="108.5602"/>
+        <inertia ixx="1.0" ixy="0.0" ixz="0.0" iyy="1.0" iyz="0.0" izz="108.5602"/>
         <mass value="8.506E2"/>
         <origin rpy="0.0 -0.0 0.0" xyz="0.1452291 0.0490361 -0.4425695"/>
