Commit message: Add ros2_control urdf files

File: create_kr240_robot_description/urdf/create_kr240_system_macro.xacro (robot description, xacro)
@@ -1,9 +1,9 @@
 <?xml version="1.0"?>
-<robot xmlns:xacro="http://www.ros.org/wiki/xacro" name="kr240_kl4000">
-    <xacro:arg name="prefix" default="" />
+<robot xmlns:xacro="http://www.ros.org/wiki/xacro" name="create_kr240_system">
+  <xacro:macro name="create_kr240_system" params="prefix">
     <xacro:include filename="$(find create_kr240_robot_description)/urdf/kr240_r3330_macro.xacro" />
     <xacro:include filename="$(find create_kr240_robot_description)/urdf/kl4000_macro.xacro" />
-    <xacro:kuka_kr240_r3330_robot prefix=""/>
-    <xacro:kuka_kl4000_rail prefix=""/>
+    <xacro:kuka_kr240_r3330_robot prefix="${prefix}"/>
+    <xacro:kuka_kl4000_rail prefix="${prefix}"/>
     <joint name="$carriage-robot" type="fixed">
       <child link="base_link"/>
@@ -11,3 +11,4 @@
       <parent link="mount"/>
     </joint>
+  </xacro:macro>
 </robot>
