Commit message: Fix URDF files

File: create_kr240_robot_description/urdf/create_kr240_system.urdf.xacro (robot description, xacro)
@@ -3,4 +3,4 @@
     <xacro:arg name="prefix" default="" />
     <xacro:include filename="$(find create_kr240_robot_description)/urdf/create_kr240_system_macro.xacro" />
-    <xacro:create_kr240_system prefix="${prefix}"/>
+    <xacro:create_kr240_system prefix="$(arg prefix)"/>
 </robot>

File: create_kr240_robot_description/urdf/create_kr240_system_macro.xacro (robot description, xacro)
@@ -5,6 +5,6 @@
     <xacro:include filename="$(find create_kr240_robot_description)/urdf/kl4000_macro.xacro" />
     <xacro:kuka_kr240_r3330_robot prefix="${prefix}"/>
-    <xacro:kuka_kl4000_rail prefix="${prefix}"/>
-    <joint name="$carriage-robot" type="fixed">
+    <xacro:kuka_kl4000_rail prefix="${prefix}" ext_axis_name="e1"/>
+    <joint name="$mount-robot" type="fixed">
       <child link="base_link"/>
       <origin rpy="0.0 0.0 0.0" xyz="0.0 0.0 0.0"/>

File: create_kr240_robot_description/urdf/kl4000_macro.xacro (robot description, xacro)
@@ -1,5 +1,5 @@
 <?xml version="1.0" encoding="UTF-8"?>
 <robot xmlns:xacro="http://www.ros.org/wiki/xacro" name="kl4000">
-  <xacro:macro name="kuka_kl4000_rail" params="prefix">
+  <xacro:macro name="kuka_kl4000_rail" params="ext_axis_name prefix">
     <!-- LINKS -->
     <!-- rail link -->
@@ -46,5 +46,5 @@
     <!-- JOINTS -->
     <!-- joint rail-carriage -->
-    <joint name="${prefix}rail-carriage" type="prismatic">
+    <joint name="${prefix}joint_${ext_axis_name}" type="prismatic">
       <axis xyz="1.0 0.0 0.0"/>
       <child link="${prefix}carriage"/>
